Commit message: Update quadcopter model.

File: data/urdf/quadcopter.urdf (robot description, URDF)
Before this commit: robot quadcopter, 1 links, 0 joints
Links:
- link base_link: geometry collision mesh filename=package://hpp-quadcopter/meshes/quadrotor_base.dae; visual mesh filename=package://hpp-quadcopter/meshes/quadrotor_base.dae
