Commit message: Update models and Python files

File: data/urdf/scene.urdf (robot description, URDF)
Before this commit: robot scene, 1 links, 0 joints
Links:
- link base_link: geometry collision mesh filename=package://hpp-quadcopter/meshes/scene.stl; visual mesh filename=package://hpp-quadcopter/meshes/scene.stl

Commit message: Add walls to the scene

File: data/urdf/scene.urdf (robot description, URDF)
Before this commit: robot scene, 1 links, 0 joints
Links:
- link base_link: geometry collision mesh filename=package://hpp-quadcopter/meshes/scene1.stl; visual mesh filename=package://hpp-quadcopter/meshes/scene1.stl

Commit message: Update scene.

File: data/urdf/scene.urdf (robot description, URDF)
Before this commit: robot scene, 1 links, 0 joints
Links:
- link base_link: geometry collision mesh filename=package://hpp-quadcopter/meshes/scene_cube.stl; collision mesh filename=package://hpp-quadcopter/meshes/scene_obs.stl
